File: cc2538node.brd (EAGLE design)
At the start: 50 x 40 mm, 44 parts, among them IC1 CC2538, IC2 MIC5225-3.3YM5, IC3 MCP73831/OT, X2 32MHz

Commit message: Cleaned up schematic and updated pdfs
Parts:
- added FRAME2: FRAME-LETTER, SparkFun-Aesthetics:CREATIVE_COMMONS
- renumbered BATT to BATT_JST, JP2 to BATT_JUMPER, JP3 to UART
Other:
- board text added: "Jelmer Tiete"
Changed lines of the file:
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@@
 <?xml version="1.0" encoding="utf-8"?>
 <!DOCTYPE eagle SYSTEM "eagle.dtd">
-<eagle version="6.5.1">
+<eagle version="7.1.0">
 <drawing>
 <settings>
@@
 <layer number="25" name="tNames" color="7" fill="1" visible="yes" active="yes"/>
 <layer number="26" name="bNames" color="7" fill="1" visible="yes" active="yes"/>
-<layer number="27" name="tValues" color="7" fill="1" visible="yes" active="yes"/>
-<layer number="28" name="bValues" color="7" fill="1" visible="yes" active="yes"/>
+<layer number="27" name="tValues" color="7" fill="1" visible="no" active="yes"/>
+<layer number="28" name="bValues" color="7" fill="1" visible="no" active="yes"/>
 <layer number="29" name="tStop" color="7" fill="3" visible="yes" active="yes"/>
 <layer number="30" name="bStop" color="7" fill="6" visible="yes" active="yes"/>
@@
 <layer number="37" name="tTest" color="7" fill="1" visible="yes" active="yes"/>
 <layer number="38" name="bTest" color="7" fill="1" visible="yes" active="yes"/>
-<layer number="39" name="tKeepout" color="4" fill="11" visible="yes" active="yes"/>
-<layer number="40" name="bKeepout" color="1" fill="11" visible="yes" active="yes"/>
-<layer number="41" name="tRestrict" color="4" fill="10" visible="yes" active="yes"/>
-<layer number="42" name="bRestrict" color="1" fill="10" visible="yes" active="yes"/>
-<layer number="43" name="vRestrict" color="2" fill="10" visible="yes" active="yes"/>
-<layer number="44" name="Drills" color="7" fill="1" visible="yes" active="yes"/>
-<layer number="45" name="Holes" color="7" fill="1" visible="yes" active="yes"/>
+<layer number="39" name="tKeepout" color="4" fill="11" visible="no" active="yes"/>
+<layer number="40" name="bKeepout" color="1" fill="11" visible="no" active="yes"/>
+<layer number="41" name="tRestrict" color="4" fill="10" visible="no" active="yes"/>
+<layer number="42" name="bRestrict" color="1" fill="10" visible="no" active="yes"/>
+<layer number="43" name="vRestrict" color="2" fill="10" visible="no" active="yes"/>
+<layer number="44" name="Drills" color="7" fill="1" visible="no" active="yes"/>
+<layer number="45" name="Holes" color="7" fill="1" visible="no" active="yes"/>
 <layer number="46" name="Milling" color="3" fill="1" visible="yes" active="yes"/>
 <layer number="47" name="Measures" color="7" fill="1" visible="yes" active="yes"/>
@@
 <layer number="56" name="wert" color="7" fill="1" visible="no" active="no"/>
 <layer number="57" name="tCAD" color="7" fill="1" visible="no" active="no"/>
+<layer number="59" name="tCarbon" color="7" fill="1" visible="no" active="no"/>
+<layer number="60" name="bCarbon" color="7" fill="1" visible="no" active="no"/>
+<layer number="90" name="Modules" color="5" fill="1" visible="no" active="no"/>
 <layer number="91" name="Nets" color="2" fill="1" visible="no" active="no"/>
 <layer number="92" name="Busses" color="1" fill="1" visible="no" active="no"/>
@@
 <layer number="97" name="Info" color="7" fill="1" visible="no" active="no"/>
 <layer number="98" name="Guide" color="6" fill="1" visible="no" active="no"/>
+<layer number="99" name="SpiceOrder" color="7" fill="1" visible="no" active="no"/>
 <layer number="100" name="Muster" color="7" fill="1" visible="no" active="no"/>
 <layer number="101" name="Patch_Top" color="12" fill="4" visible="yes" active="yes"/>
@@
 <layer number="127" name="_tValues" color="7" fill="1" visible="yes" active="yes"/>
 <layer number="128" name="_bValues" color="7" fill="1" visible="yes" active="yes"/>
+<layer number="129" name="Mask" color="7" fill="1" visible="yes" active="yes"/>
 <layer number="131" name="prix" color="7" fill="1" visible="yes" active="yes"/>
 <layer number="132" name="test" color="7" fill="1" visible="yes" active="yes"/>
@@
 <layer number="223" name="223bmp" color="24" fill="1" visible="no" active="no"/>
 <layer number="224" name="224bmp" color="25" fill="1" visible="no" active="no"/>
+<layer number="225" name="225bmp" color="7" fill="1" visible="yes" active="yes"/>
+<layer number="226" name="226bmp" color="7" fill="1" visible="yes" active="yes"/>
+<layer number="227" name="227bmp" color="7" fill="1" visible="yes" active="yes"/>
+<layer number="228" name="228bmp" color="7" fill="1" visible="yes" active="yes"/>
+<layer number="229" name="229bmp" color="7" fill="1" visible="yes" active="yes"/>
+<layer number="230" name="230bmp" color="7" fill="1" visible="yes" active="yes"/>
+<layer number="231" name="231bmp" color="7" fill="1" visible="yes" active="yes"/>
 <layer number="248" name="Housing" color="7" fill="1" visible="yes" active="yes"/>
 <layer number="249" name="Edge" color="7" fill="1" visible="yes" active="yes"/>
@@
 <layer number="251" name="SMDround" color="12" fill="11" visible="no" active="no"/>
 <layer number="254" name="cooling" color="7" fill="1" visible="yes" active="yes"/>
+<layer number="255" name="routoute" color="7" fill="1" visible="yes" active="yes"/>
 </layers>
 <board>
@@
 <dimension x1="0" y1="0" x2="0" y2="40" x3="-6" y3="20" textsize="1.778" layer="47"/>
 <dimension x1="0" y1="40" x2="50" y2="40" x3="25" y3="44.8" textsize="1.778" layer="47"/>
+<text x="21.8" y="-18.4" size="1.778" layer="51">Jelmer Tiete</text>
 </plain>
 <attributes>
@@
 <pass name="Default">
 <param name="RoutingGrid" value="50mil"/>
+<param name="AutoGrid" value="1"/>
+<param name="Efforts" value="0"/>
+<param name="TopRouterVariant" value="1"/>
 <param name="tpViaShape" value="round"/>
 <param name="PrefDir.1" value="|"/>
@@
 <attribute name="VALUE" x="15.27" y="11.905" size="0.4064" layer="27" rot="R180"/>
 </element>
-<element name="BATT" library="adafruit" package="JST-PH-2-SMT-RA" value="" x="6.1" y="9" smashed="yes" rot="R90">
+<element name="BATT_JST" library="adafruit" package="JST-PH-2-SMT-RA" value="" x="6.1" y="9" smashed="yes" rot="R90">
 <attribute name="NAME" x="3.56" y="13.51" size="1.27" layer="25" font="vector"/>
 <attribute name="VALUE" x="13.72" y="6.46" size="1.27" layer="27" font="vector" rot="R90"/>
 </element>
-<element name="JP2" library="SparkFun-Connectors" package="1X02_LONGPADS" value="M02PTH3" x="5.3" y="10.305" rot="R270"/>
+<element name="BATT_JUMPER" library="SparkFun-Connectors" package="1X02_LONGPADS" value="M02PTH3" x="5.3" y="10.305" rot="R270"/>
 <element name="C1" library="dp_devices" package="C603" value="1.0uF" x="31.8" y="24" smashed="yes">
 <attribute name="NAME" x="30.83" y="22.0525" size="1.27" layer="25" ratio="10"/>
@@
 <attribute name="VALUE" x="14.0775" y="21.57" size="1.27" layer="27" ratio="10" rot="R270"/>
 </element>
-<element name="JP3" library="SparkFun-Connectors" package="1X03_NO_SILK" value="" x="47.9" y="11.5" smashed="yes" rot="R270">
+<element name="UART" library="SparkFun-Connectors" package="1X03_NO_SILK" value="" x="47.9" y="11.5" smashed="yes" rot="R270">
 <attribute name="VALUE" x="44.725" y="12.77" size="1.27" layer="27" rot="R270"/>
 </element>
@@
 <attribute name="VALUE" x="21.24" y="17.5225" size="1.27" layer="27" ratio="10" rot="R180"/>
 </element>
+<element name="FRAME2" library="SparkFun-Aesthetics" package="CREATIVE_COMMONS" value="FRAME-LETTER" x="-9" y="-18.4"/>
 </elements>
 <signals>
@@
 <contactref element="IC2" pad="2"/>
 <contactref element="IC3" pad="2"/>
-<contactref element="BATT" pad="2"/>
+<contactref element="BATT_JST" pad="2"/>
 <contactref element="C1" pad="2"/>
 <contactref element="R1" pad="2"/>
@@
 <contactref element="C6" pad="2"/>
 <contactref element="C8" pad="2"/>
-<contactref element="JP2" pad="2"/>
+<contactref element="BATT_JUMPER" pad="2"/>
 <contactref element="R5" pad="2"/>
 <contactref element="C11" pad="2"/>
@@
 <contactref element="U$3" pad="19"/>
 <contactref element="U$3" pad="1"/>
-<contactref element="JP3" pad="1"/>
+<contactref element="UART" pad="1"/>
 <wire x1="26" y1="17.8" x2="26" y2="18.7" width="0.3048" layer="1"/>
 <polygon width="0.2" layer="16">
@@
 <contactref element="IC3" pad="3"/>
 <contactref element="SJ1" pad="3"/>
-<contactref element="BATT" pad="1"/>
-<contactref element="JP2" pad="1"/>
+<contactref element="BATT_JST" pad="1"/>
+<contactref element="BATT_JUMPER" pad="1"/>
 <contactref element="C15" pad="1"/>
 <wire x1="5.7" y1="26.05" x2="5.7" y2="25.9" width="0.4064" layer="1"/>
@@
 <signal name="RXD">
 <contactref element="IC1" pad="16"/>
-<contactref element="JP3" pad="2"/>
+<contactref element="UART" pad="2"/>
 <wire x1="30" y1="16.85" x2="30.9" y2="16.85" width="0.3048" layer="1"/>
 <wire x1="30.9" y1="16.85" x2="32.15" y2="15.6" width="0.3048" layer="1"/>
@@
 <signal name="TXD">
 <contactref element="IC1" pad="17"/>
-<contactref element="JP3" pad="3"/>
+<contactref element="UART" pad="3"/>
 <wire x1="30" y1="17.35" x2="31.8" y2="17.35" width="0.3048" layer="1"/>
 <wire x1="31.8" y1="17.35" x2="32.85" y2="16.3" width="0.3048" layer="1"/>
