File: cc2538node.sch (EAGLE design)
At the start: 44 parts, among them IC1 CC2538, IC2 MIC5225-3.3YM5, IC3 MCP73831/OT, X2 32MHz

Commit message: Cleaned up schematic and updated pdfs
Parts:
- removed BATT: (no value), adafruit:JST_2PIN-SMT-RA
- removed JP2: M02PTH3, SparkFun-Connectors:M02PTH3
- removed JP3: (no value), SparkFun-Connectors:M031X03_NO_SILK
- added BATT_JST: (no value), adafruit:JST_2PIN-SMT-RA
- added BATT_JUMPER: M02PTH3, SparkFun-Connectors:M02PTH3
- added FRAME2: FRAME-LETTER, SparkFun-Aesthetics:FRAME-LETTER
- added UART: (no value), SparkFun-Connectors:M031X03_NO_SILK
Connections:
- net GND: now also BATT_JST.1, BATT_JUMPER.2, UART.1; no longer BATT.1, JP2.2, JP3.1
- net RXD: now also UART.2; no longer JP3.2
- net TXD: now also UART.3; no longer JP3.3
- net V_BATT: now also BATT_JST.2, BATT_JUMPER.1; no longer BATT.2, JP2.1
Other:
- note added: "1.0"
- note added: "CC2538"
- note added: "I/O"
- note added: "Jelmer Tiete"
- note added: "Power supply and battery charger"
- note removed: "(C) Jelmer Tiete 2014"
- moved on the sheet: BTN1, C1, C10, C11, C12, C13, C14, C15, C16, C17, C18, C3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
